File: UltrasonicTRSwitch_Tester.kicad_pcb (KiCad board)
At the start: 4 copper layers, 89 x 54.2 mm, 60 parts, among them IC1 MAX4937CTN+, IC2 MIC5270-5.0YM5_TR, J1 Conn_01x01_Female, J10 Conn_01x01_Female, J11 Conn_01x01_Female, J12 Conn_01x01_Female, J13 Conn_01x01_Female, J14 Conn_01x01_Female, J15 Conn_01x01_Female, J16 Conn_01x01_Female, J17 Conn_01x02_Female, J18 Conn_01x02_Female, J19 Conn_01x05_Female, J2 Conn_01x01_Female, J20 Conn_01x01_Female, J21 Conn_01x01_Female, J22 Conn_01x01_Female, J23 Conn_01x01_Female, J24 Conn_01x01_Female, J25 Conn_01x01_Female, J26 Conn_01x01_Female, J27 Conn_01x01_Female, J3 Conn_01x01_Female, J4 Conn_01x01_Female, J5 Conn_01x01_Female, J6 Conn_01x01_Female, J7 Conn_01x01_Female, J8 Conn_01x01_Female, J9 Conn_01x01_Female, U1 MIC5205-5.0YM5, U2 MIC5501-3.0YM5

Commit message: Updated footprints and board size
Parts:
- moved J17 21.6 mm to (102.0, 43.5)
- moved J18 18.1 mm to (84.5, 43.5)
- moved H4 10.8 mm to (100.0, 20.0)
- moved H2 10.3 mm to (100.0, 68.0)
- moved H3 2.30 mm to (10.0, 68.0)
- moved H1 1.77 mm to (10.0, 20.0)
Routing:
- net GND: track 31.6 -> 45.3 mm, vias 58 -> 59
- net +10V: track 32.4 -> 43.8 mm
- net -10V: track 11.2 -> 21.6 mm
Other:
- board size 89 x 54.2 mm -> 106.2 x 54.2 mm
